Commit message: small bug fixes to urdfs

File: sim_ws/src/nav2_gps_waypoint_follower_demo/urdf/wheel_module_macro.xacro (robot description, xacro)
@@ -15,5 +15,5 @@
         - side: left or right
     -->
-    <xacro:macro name="wheel_assembly" params="parent_name mass radius width module_len cx cy cz side">
+    <xacro:macro name="wheel_assembly" params="parent_name mass radius width module_len module_width_x module_width_y cx cy cz side">
         <!--
         Firstly create a link for the wheel module
@@ -22,11 +22,9 @@
         Then create a joint to connect the wheel to the wheel module
         -->
-        <joint name="joint_steering_to_wheel_${name}" type="continuous">
+        <joint name="wheel_module_${parent_name}_joint" type="continuous">
             <parent link="${parent_name}"/>
             <child link="$wheel_module_{parent_name}"/>
             <origin xyz="${cx} ${cy} ${cz}" rpy="0 0 0"/> <!--This origin is where child link is placed w.r.t parent link -->
         </joint>
-        <xacro:property name="module_width_y" value="0.15"/> <!-- Width of arm along y axis -->
-        <xacro:property name="module_width_x" value="0.2"/> <!-- Width of arm along x axis -->
         <!-- Define the wheel module link -->
         <link name="wheel_module_${parent_name}">
@@ -49,5 +47,5 @@
         </link>
         <!-- Define the wheel link -->
-        <joint name="wheel_${parent_name}" type="continuous">
+        <joint name="wheel_${parent_name}_joint" type="continuous">
             <parent link="wheel_module_${parent_name}"/>
             <child link="wheel_${parent_name}"/>

File: sim_ws/src/simulation_launch/description/robot.urdf.xacro (robot description, xacro)
@@ -17,6 +17,6 @@
     <xacro:property name="base_to_module_x" value="1.2" /> <!-- meters -->
     <xacro:property name="base_to_module_y" value="0.6" />
-    <xacro:property name="module_len_x" value="0.2" />
-    <xacro:property name="module_len_y" value="0.15" />
+    <xacro:property name="module_width_x" value="0.2" />
+    <xacro:property name="module_width_y" value="0.15" />
     <xacro:property name="module_height" value="0.8" />
     <!-- Wheel dimensions -->
@@ -70,9 +70,9 @@
     </joint>
     <!-- Define the wheel modules -->
-    <!-- params="parent_name mass radius width module_len cx cy cz side" -->
+    <!-- params="parent_name mass radius width module_len module_width_x module_width_y cx cy cz side" -->
     <!-- NOTE: cx,cy,cz are the coordinates of the child link's center w.r.t the parent link -->
-    <xacro:wheel_assembly parent_name="front_left" mass="${wheel_mass}" radius="${wheel_radius}" width="${wheel_width}" module_len="${module_height}" cx="0" cy="0" cz="-${module_height}/2" side="left"/>
-    <xacro:wheel_assembly parent_name="front_right" mass="${wheel_mass}" radius="${wheel_radius}" width="${wheel_width}" module_len="${module_height}" cx="0" cy="0" cz="-${module_height}/2" side="right"/>
-    <xacro:wheel_assembly parent_name="rear_left" mass="${wheel_mass}" radius="${wheel_radius}" width="${wheel_width}" module_len="${module_height}" cx="0" cy="0" cz="-${module_height}/2" side="left"/>
-    <xacro:wheel_assembly parent_name="rear_right" mass="${wheel_mass}" radius="${wheel_radius}" width="${wheel_width}" module_len="${module_height}" cx="0" cy="0" cz="-${module_height}/2" side="right"/>
+    <xacro:wheel_assembly parent_name="front_left" mass="${wheel_mass}" radius="${wheel_radius}" width="${wheel_width}" module_len="${module_height}" module_width_x="${module_width_x}" module_width_y="${module_width_y}" cx="0" cy="0" cz="-${module_height}/2" side="left"/>
+    <xacro:wheel_assembly parent_name="front_right" mass="${wheel_mass}" radius="${wheel_radius}" width="${wheel_width}" module_len="${module_height}" module_width_x="${module_width_x}" module_width_y="${module_width_y}" cx="0" cy="0" cz="-${module_height}/2" side="right"/>
+    <xacro:wheel_assembly parent_name="rear_left" mass="${wheel_mass}" radius="${wheel_radius}" width="${wheel_width}" module_len="${module_height}" module_width_x="${module_width_x}" module_width_y="${module_width_y}" cx="0" cy="0" cz="-${module_height}/2" side="left"/>
+    <xacro:wheel_assembly parent_name="rear_right" mass="${wheel_mass}" radius="${wheel_radius}" width="${wheel_width}" module_len="${module_height}" module_width_x="${module_width_x}" module_width_y="${module_width_y}" cx="0" cy="0" cz="-${module_height}/2" side="right"/>
 </robot>

File: sim_ws/src/simulation_launch/description/wheel_module_macro.xacro (robot description, xacro)
@@ -15,5 +15,5 @@
         - side: left or right
     -->
-    <xacro:macro name="wheel_assembly" params="parent_name mass radius width module_len cx cy cz side">
+    <xacro:macro name="wheel_assembly" params="parent_name mass radius width module_len module_width_x module_width_y cx cy cz side">
         <!--
         Firstly create a link for the wheel module
@@ -22,15 +22,13 @@
         Then create a joint to connect the wheel to the wheel module
         -->
-        <joint name="joint_steering_to_wheel_${name}" type="continuous">
+        <joint name="wheel_module_${parent_name}_joint" type="continuous">
             <parent link="${parent_name}"/>
             <child link="$wheel_module_{parent_name}"/>
             <origin xyz="${cx} ${cy} ${cz}" rpy="0 0 0"/> <!--This origin is where child link is placed w.r.t parent link -->
         </joint>
-        <xacro:property name="module_width_y" value="0.15"/> <!-- Width of arm along y axis -->
-        <xacro:property name="module_width_x" value="0.2"/> <!-- Width of arm along x axis -->
         <!-- Define the wheel module link -->
         <link name="wheel_module_${parent_name}">
             <visual>
-                <origin xyz="0 0 -${module_len}/2"/> <!--This origin is w.r.t the wheel_module_${parent_name} link -->
+                <origin xyz="0 0 0"/> <!--This origin is w.r.t the wheel_module_${parent_name} link -->
                 <geometry>
                     <box size="module_width_x module_width_y ${module_len}"/>
@@ -39,5 +37,5 @@
             </visual>
             <collision>
-                <origin xyz="0 0 -${module_len}/2"/> <!--This origin is w.r.t the wheel_module_${parent_name} link -->
+                <origin xyz="0 0 0"/> <!--This origin is w.r.t the wheel_module_${parent_name} link -->
                 <geometry>
                     <box size="module_width_x module_width_y ${module_len}"/>
@@ -45,12 +43,12 @@
             </collision>
             <xacro:inertial_box mass="0.5" x="module_width_x" y="module_width_y" z="${module_len}">
-                <origin xyz="0 0 -${module_len}/2" rpy="0 0 0"/>
+                <origin xyz="0 0 0" rpy="0 0 0"/>
             </xacro:inertial_box>
         </link>
         <!-- Define the wheel link -->
-        <joint name="wheel_${parent_name}" type="continuous">
+        <joint name="wheel_${parent_name}_joint" type="continuous">
             <parent link="wheel_module_${parent_name}"/>
             <child link="wheel_${parent_name}"/>
-            <origin xyz="0 $(if ${side} == 'left', '-${width}', '${width}') -${module_len}/2" rpy="0 0 $(if ${side} == 'left', '-${pi/2}', '${pi/2}')"/>
+            <origin xyz="0 $(if ${side} == 'left', '${width}', '-${width}') -${module_len}/2" rpy="0 0 $(if ${side} == 'left', '-${pi/2}', '${pi/2}')"/>
             <axis xyz="0 0 1"/>
         </joint>

Commit message: bug fixes in urdf

File: sim_ws/src/nav2_gps_waypoint_follower_demo/urdf/wheel_module_macro.xacro (robot description, xacro)
@@ -24,5 +24,5 @@
         <joint name="wheel_module_${parent_name}_joint" type="continuous">
             <parent link="${parent_name}"/>
-            <child link="$wheel_module_{parent_name}"/>
+            <child link="wheel_module_${parent_name}"/>
             <origin xyz="${cx} ${cy} ${cz}" rpy="0 0 0"/> <!--This origin is where child link is placed w.r.t parent link -->
         </joint>
@@ -32,5 +32,5 @@
                 <origin xyz="0 0 0"/> <!--This origin is w.r.t the wheel_module_${parent_name} link -->
                 <geometry>
-                    <box size="module_width_x module_width_y ${module_len}"/>
+                    <box size="${module_width_x} ${module_width_y} ${module_len}"/>
                 </geometry>
                 <material name="grey"/>
@@ -39,16 +39,25 @@
                 <origin xyz="0 0 0"/> <!--This origin is w.r.t the wheel_module_${parent_name} link -->
                 <geometry>
-                    <box size="module_width_x module_width_y ${module_len}"/>
+                    <box size="${module_width_x} ${module_width_y} ${module_len}"/>
                 </geometry>
             </collision>
-            <xacro:inertial_box mass="0.5" x="module_width_x" y="module_width_y" z="${module_len}">
+            <!-- !Hardcoded mass -->
+            <xacro:inertial_box mass="2.0" x="${module_width_x}" y="${module_width_y}" z="${module_len}">
                 <origin xyz="0 0 0" rpy="0 0 0"/>
             </xacro:inertial_box>
         </link>
         <!-- Define the wheel link -->
+        <xacro:if value="${side == 'left'}">
+            <xacro:property name="wheel_position_y" value="-${width}"/>
+            <xacro:property name="wheel_rpy" value="-${PI/2}"/>
+        </xacro:if>
+        <xacro:if value="${side == 'right'}">
+            <xacro:property name="wheel_position_y" value="${width}"/>
+            <xacro:property name="wheel_rpy" value="${PI/2}"/>
+        </xacro:if>
         <joint name="wheel_${parent_name}_joint" type="continuous">
             <parent link="wheel_module_${parent_name}"/>
             <child link="wheel_${parent_name}"/>
-            <origin xyz="0 $(if ${side} == 'left', '${width}', '-${width}') -${module_len}/2" rpy="0 0 $(if ${side} == 'left', '-${pi/2}', '${pi/2}')"/>
+            <origin xyz="0 ${wheel_position_y} -${module_len}/2" rpy="0 0 ${wheel_yaw}"/>
             <axis xyz="0 0 1"/>
         </joint>

File: sim_ws/src/simulation_launch/description/robot.urdf.xacro (robot description, xacro)
@@ -72,7 +72,7 @@
     <!-- params="parent_name mass radius width module_len module_width_x module_width_y cx cy cz side" -->
     <!-- NOTE: cx,cy,cz are the coordinates of the child link's center w.r.t the parent link -->
-    <xacro:wheel_assembly parent_name="front_left" mass="${wheel_mass}" radius="${wheel_radius}" width="${wheel_width}" module_len="${module_height}" module_width_x="${module_width_x}" module_width_y="${module_width_y}" cx="0" cy="0" cz="-${module_height}/2" side="left"/>
-    <xacro:wheel_assembly parent_name="front_right" mass="${wheel_mass}" radius="${wheel_radius}" width="${wheel_width}" module_len="${module_height}" module_width_x="${module_width_x}" module_width_y="${module_width_y}" cx="0" cy="0" cz="-${module_height}/2" side="right"/>
-    <xacro:wheel_assembly parent_name="rear_left" mass="${wheel_mass}" radius="${wheel_radius}" width="${wheel_width}" module_len="${module_height}" module_width_x="${module_width_x}" module_width_y="${module_width_y}" cx="0" cy="0" cz="-${module_height}/2" side="left"/>
-    <xacro:wheel_assembly parent_name="rear_right" mass="${wheel_mass}" radius="${wheel_radius}" width="${wheel_width}" module_len="${module_height}" module_width_x="${module_width_x}" module_width_y="${module_width_y}" cx="0" cy="0" cz="-${module_height}/2" side="right"/>
+    <xacro:wheel_assembly parent_name="front_left" mass="${wheel_mass}" radius="${wheel_radius}" width="${wheel_width}" module_len="${module_height}" module_width_x="${module_width_x}" module_width_y="${module_width_y}" cx="0" cy="0" cz="${-module_height/2.0}" side="left"/>
+    <xacro:wheel_assembly parent_name="front_right" mass="${wheel_mass}" radius="${wheel_radius}" width="${wheel_width}" module_len="${module_height}" module_width_x="${module_width_x}" module_width_y="${module_width_y}" cx="0" cy="0" cz="${-module_height/2.0}" side="right"/>
+    <xacro:wheel_assembly parent_name="rear_left" mass="${wheel_mass}" radius="${wheel_radius}" width="${wheel_width}" module_len="${module_height}" module_width_x="${module_width_x}" module_width_y="${module_width_y}" cx="0" cy="0" cz="${-module_height/2.0}" side="left"/>
+    <xacro:wheel_assembly parent_name="rear_right" mass="${wheel_mass}" radius="${wheel_radius}" width="${wheel_width}" module_len="${module_height}" module_width_x="${module_width_x}" module_width_y="${module_width_y}" cx="0" cy="0" cz="${-module_height/2.0}" side="right"/>
 </robot>

File: sim_ws/src/simulation_launch/description/wheel_module_macro.xacro (robot description, xacro)
@@ -24,5 +24,5 @@
         <joint name="wheel_module_${parent_name}_joint" type="continuous">
             <parent link="${parent_name}"/>
-            <child link="$wheel_module_{parent_name}"/>
+            <child link="wheel_module_${parent_name}"/>
             <origin xyz="${cx} ${cy} ${cz}" rpy="0 0 0"/> <!--This origin is where child link is placed w.r.t parent link -->
         </joint>
@@ -32,5 +32,5 @@
                 <origin xyz="0 0 0"/> <!--This origin is w.r.t the wheel_module_${parent_name} link -->
                 <geometry>
-                    <box size="module_width_x module_width_y ${module_len}"/>
+                    <box size="${module_width_x} ${module_width_y} ${module_len}"/>
                 </geometry>
                 <material name="grey"/>
@@ -39,16 +39,25 @@
                 <origin xyz="0 0 0"/> <!--This origin is w.r.t the wheel_module_${parent_name} link -->
                 <geometry>
-                    <box size="module_width_x module_width_y ${module_len}"/>
+                    <box size="${module_width_x} ${module_width_y} ${module_len}"/>
                 </geometry>
             </collision>
-            <xacro:inertial_box mass="0.5" x="module_width_x" y="module_width_y" z="${module_len}">
+            <!-- !Hardcoded mass -->
+            <xacro:inertial_box mass="2.0" x="${module_width_x}" y="${module_width_y}" z="${module_len}">
                 <origin xyz="0 0 0" rpy="0 0 0"/>
             </xacro:inertial_box>
         </link>
         <!-- Define the wheel link -->
+        <xacro:if value="${side == 'left'}">
+            <xacro:property name="wheel_position_y" value="-${width}"/>
+            <xacro:property name="wheel_yaw" value="-${PI/2}"/>
+        </xacro:if>
+        <xacro:if value="${side == 'right'}">
+            <xacro:property name="wheel_position_y" value="${width}"/>
+            <xacro:property name="wheel_yaw" value="${PI/2}"/>
+        </xacro:if>
         <joint name="wheel_${parent_name}_joint" type="continuous">
             <parent link="wheel_module_${parent_name}"/>
             <child link="wheel_${parent_name}"/>
-            <origin xyz="0 $(if ${side} == 'left', '${width}', '-${width}') -${module_len}/2" rpy="0 0 $(if ${side} == 'left', '-${pi/2}', '${pi/2}')"/>
+            <origin xyz="0 ${wheel_position_y} -${module_len}/2" rpy="0 0 ${wheel_yaw}"/>
             <axis xyz="0 0 1"/>
         </joint>

Commit message: urdf finally has right syntax

File: sim_ws/src/nav2_gps_waypoint_follower_demo/urdf/wheel_module_macro.xacro (robot description, xacro)
@@ -1,6 +1,6 @@
 <?xml version="1.0" ?>
 <robot xmlns:xacro="http://www.ros.org/wiki/xacro" >
-    <include filename="$(find nav2_gps_waypoint_follower_demo)/urdf/color_macro.xacro"/>
-    <inclue filename = "$(find nav2_gps_waypoint_follower_demo)/urdf/inertia_macro.xacro"/>
+    <include filename="color_macro.xacro"/>
+    <include filename="inertia_macro.xacro"/>
     <!--
         A macro to create a wheel module (including links and joints)
@@ -50,14 +50,14 @@
         <xacro:if value="${side == 'left'}">
             <xacro:property name="wheel_position_y" value="-${width}"/>
-            <xacro:property name="wheel_rpy" value="-${PI/2}"/>
+            <xacro:property name="wheel_yaw" value="-${PI/2}"/>
         </xacro:if>
         <xacro:if value="${side == 'right'}">
             <xacro:property name="wheel_position_y" value="${width}"/>
-            <xacro:property name="wheel_rpy" value="${PI/2}"/>
+            <xacro:property name="wheel_yaw" value="${PI/2}"/>
         </xacro:if>
         <joint name="wheel_${parent_name}_joint" type="continuous">
             <parent link="wheel_module_${parent_name}"/>
             <child link="wheel_${parent_name}"/>
-            <origin xyz="0 ${wheel_position_y} -${module_len}/2" rpy="0 0 ${wheel_yaw}"/>
+            <origin xyz="0 ${wheel_position_y} ${-module_len/2.0}" rpy="0 0 ${wheel_yaw}"/>
             <axis xyz="0 0 1"/>
         </joint>

File: sim_ws/src/simulation_launch/description/wheel_module_macro.xacro (robot description, xacro)
@@ -1,6 +1,6 @@
 <?xml version="1.0" ?>
 <robot xmlns:xacro="http://www.ros.org/wiki/xacro" >
-    <include filename="$(find nav2_gps_waypoint_follower_demo)/urdf/color_macro.xacro"/>
-    <inclue filename = "$(find nav2_gps_waypoint_follower_demo)/urdf/inertia_macro.xacro"/>
+    <include filename="color_macro.xacro"/>
+    <include filename="inertia_macro.xacro"/>
     <!--
         A macro to create a wheel module (including links and joints)
@@ -59,5 +59,5 @@
             <parent link="wheel_module_${parent_name}"/>
             <child link="wheel_${parent_name}"/>
-            <origin xyz="0 ${wheel_position_y} -${module_len}/2" rpy="0 0 ${wheel_yaw}"/>
+            <origin xyz="0 ${wheel_position_y} ${-module_len/2.0}" rpy="0 0 ${wheel_yaw}"/>
             <axis xyz="0 0 1"/>
         </joint>

Commit message: syntax changes (not functional)

File: sim_ws/src/nav2_gps_waypoint_follower_demo/urdf/wheel_module_macro.xacro (robot description, xacro)
@@ -67,5 +67,5 @@
                     <cylinder radius="${radius}" length="${width}"/>
                 </geometry>
-                <material name="dark"/>
+                <material name="grey"/>
             </visual>
             <collision>

File: sim_ws/src/simulation_launch/description/robot.urdf.xacro (robot description, xacro)
@@ -1,4 +1,4 @@
 <?xml version="1.0"?>
-<robot xmlns:xacro="http://www.ros.org/wiki/xacro"  name="robot">
+<robot xmlns:xacro="http://www.ros.org/wiki/xacro" name="robot">
     <!-- <xacro:include filename="robot_core.xacro" /> -->
     <!-- REFER TO IMAGES FOLDER FOR VISUAL REPRESENTATION OF THE ROBOT -->
@@ -10,22 +10,31 @@
     <!-- <xacro:arg name="is_simulation" default="true" /> -->
     <!-- Chassis dimensions -->
-    <xacro:property name="chassis_mass" value="30.0" /> <!-- kilograms -->
-    <xacro:property name="chassis_length" value="3" /> <!-- meters -->
-    <xacro:property name="chassis_width" value="1.5" />
-    <xacro:property name="chassis_height" value="0.3" />
+    <xacro:property name="chassis_mass" value="30.0"/> <!-- kilograms -->
+    <xacro:property name="chassis_length" value="3"/> <!-- meters -->
+    <xacro:property name="chassis_width" value="1.5"/>
+    <xacro:property name="chassis_height" value="0.3"/>
     <!-- Wheel Module dimensions -->
-    <xacro:property name="base_to_module_x" value="1.2" /> <!-- meters -->
-    <xacro:property name="base_to_module_y" value="0.6" />
-    <xacro:property name="module_width_x" value="0.2" />
-    <xacro:property name="module_width_y" value="0.15" />
-    <xacro:property name="module_height" value="0.8" />
+    <xacro:property name="base_to_module_x" value="1.2"/> <!-- meters -->
+    <xacro:property name="base_to_module_y" value="0.6"/>
+    <xacro:property name="module_width_x" value="0.2"/>
+    <xacro:property name="module_width_y" value="0.15"/>
+    <xacro:property name="module_height" value="0.8"/>
     <!-- Wheel dimensions -->
-    <xacro:property name="wheel_mass" value="1.0" /> <!-- kilograms -->
-    <xacro:property name="wheel_radius" value="0.3" /> <!-- meters -->
-    <xacro:property name="wheel_width" value="0.1" />
+    <xacro:property name="wheel_mass" value="1.0"/> <!-- kilograms -->
+    <xacro:property name="wheel_radius" value="0.3"/> <!-- meters -->
+    <xacro:property name="wheel_width" value="0.1"/>
     <!-- Define a base link for the robot -->
     <link name="base_link">
+    </link>
+    <!-- Define a chassis link for the robot -->
+    <joint name="chassis_joint" type="fixed">
+        <parent link="base_link"/>
+        <child link="chassis"/>
+        Place the chassis at half of chassis height above the base link
+        <origin xyz="0 0 ${chassis_height/2.0}" rpy="0 0 0"/>
+    </joint>
+    <link name="chassis">
         <visual>
-            <origin xyz="0 0 0" rpy="0 0 0"/>
+            <origin xyz="0 0 0"/>
             <geometry>
                 <box size="${chassis_length} ${chassis_width} ${chassis_height}"/>
@@ -34,5 +43,5 @@
         </visual>
         <collision>
-            <origin xyz="0 0 0" rpy="0 0 0"/>
+            <origin xyz="0 0 0"/>
             <geometry>
                 <box size="${chassis_length} ${chassis_width} ${chassis_height}"/>
@@ -42,10 +51,4 @@
             <origin xyz="0 0 0" rpy="0 0 0"/>
         </xacro:inertial_box>
-    </link>
-    <!-- Define 4 static links which will be used to connect the wheel modules to the base link -->
-    <link name="front_left"> </link>
-    <link name="front_right"> </link>
-    <link name="rear_left"> </link>
-    <link name="rear_right"> </link>
     <!-- Define joints to connect static links to the base link -->
     <joint name="FL_joint" type="fixed">
@@ -69,4 +72,13 @@
         <origin xyz="-${base_to_module_x} -${base_to_module_y} 0" rpy="0 0 0"/>
     </joint>
+    <!-- Define 4 static links which will be used to connect the wheel modules to the base link -->
+    <link name="front_left">
+    </link>
+    <link name="front_right">
+    </link>
+    <link name="rear_left">
+    </link>
+    <link name="rear_right">
+    </link>
     <!-- Define the wheel modules -->
     <!-- params="parent_name mass radius width module_len module_width_x module_width_y cx cy cz side" -->
