Commit message: added base_footprint frame and ensured robot above ground plane

File: sim_ws/src/nav2_gps_waypoint_follower_demo/urdf/robot.urdf.xacro (robot description, xacro)
@@ -24,7 +24,12 @@
     <xacro:property name="wheel_radius" value="0.3"/> <!-- meters -->
     <xacro:property name="wheel_width" value="0.1"/>
-    <!-- Define a base link for the robot -->
-    <link name="base_link">
-    </link>
+    <!-- Define a base links for the robot. base_link and base_footprint needed for Nav2 -->
+    <link name="base_footprint"/>
+    <joint name="base_joint" type="fixed">
+        <parent link="base_footprint"/>
+        <child link="base_link"/>
+        <origin xyz="0 0 ${module_height + wheel_radius}" rpy="0 0 0"/>
+    </joint>
+    <link name="base_link"/>
     <!-- Define a chassis link for the robot -->
     <joint name="chassis_joint" type="fixed">

Commit message: started working on updated sdf

File: sim_ws/src/nav2_gps_waypoint_follower_demo/urdf/robot.urdf.xacro (robot description, xacro)
@@ -94,3 +94,45 @@
     <xacro:wheel_assembly parent_name="rear_left" mass="${wheel_mass}" radius="${wheel_radius}" width="${wheel_width}" module_len="${module_height}" module_width_x="${module_width_x}" module_width_y="${module_width_y}" cx="0" cy="0" cz="${-module_height/2.0}" side="left"/>
     <xacro:wheel_assembly parent_name="rear_right" mass="${wheel_mass}" radius="${wheel_radius}" width="${wheel_width}" module_len="${module_height}" module_width_x="${module_width_x}" module_width_y="${module_width_y}" cx="0" cy="0" cz="${-module_height/2.0}" side="right"/>
+    <!-- IMU temporarily placed 5cm above base link -->
+    <joint name="imu_joint" type="fixed">
+        <parent link="base_link"/>
+        <child link="imu_link"/>
+        <origin xyz="0.0 0.0 ${chassis_height/3}" rpy="0 0 0"/>
+    </joint>
+    <link name="imu_link"/>
+    <!-- GPS link at base link -->
+    <joint name="gps_joint" type="fixed">
+        <parent link="base_link"/>
+        <child link="gps_link"/>
+        <origin xyz="0 0 0" rpy="0 0 0"/>
+    </joint>
+    <link name="gps_link"/>
+    <!-- 2D Lidar placed in front center 20cm below chassis-->
+    <joint name="scan_joint" type="fixed">
+        <parent link="base_link"/>
+        <child link="base_scan"/>
+        <origin xyz="${chassis_length/2} 0 -0.2" rpy="0 0 0"/>
+    </joint>
+    <link name="base_scan">
+        <visual>
+        <origin xyz="0 0 0" rpy="0 0 0"/>
+        <geometry>
+            <mesh filename="package://turtlebot3_gazebo/models/turtlebot3_common/meshes/lds.dae" scale="0.001 0.001 0.001"/>
+        </geometry>
+        <material name="dark"/>
+        </visual>
+        <collision>
+        <origin xyz="0.015 0 -0.0065" rpy="0 0 0"/>
+        <geometry>
+            <cylinder length="0.0315" radius="0.055"/>
+        </geometry>
+        </collision>
+        <inertial>
+        <mass value="0.114" />
+        <origin xyz="0 0 0" />
+        <inertia ixx="0.001" ixy="0.0" ixz="0.0"
+                iyy="0.001" iyz="0.0"
+                izz="0.001" />
+        </inertial>
+    </link>
 </robot>
