Commit message: trying to add acron instead of turtlebot

File: sim_ws/src/nav2_gps_waypoint_follower_demo/urdf/acorn.xacro (robot description, xacro)
@@ -1,4 +1,4 @@
 <?xml version="1.0"?>
-<robot xmlns:xacro="http://www.ros.org/wiki/xacro" name="robot">
+<robot xmlns:xacro="http://www.ros.org/wiki/xacro" name="acron">
     <!-- <xacro:include filename="robot_core.xacro" /> -->
     <!-- REFER TO IMAGES FOLDER FOR VISUAL REPRESENTATION OF THE ROBOT -->
@@ -117,7 +117,4 @@
         <visual>
         <origin xyz="0 0 0" rpy="0 0 0"/>
-        <geometry>
-            <mesh filename="package://turtlebot3_gazebo/models/turtlebot3_common/meshes/lds.dae" scale="0.001 0.001 0.001"/>
-        </geometry>
         <material name="dark"/>
         </visual>
@@ -136,3 +133,5 @@
         </inertial>
     </link>
+    <!-- Include gazebo macros for sim -->
+    <xacro:include filename="gazebo_macro.xacro" />
 </robot>

File: sim_ws/src/nav2_gps_waypoint_follower_demo/urdf/wheel_module_macro.xacro (robot description, xacro)
@@ -26,4 +26,6 @@
             <child link="wheel_module_${parent_name}"/>
             <origin xyz="${cx} ${cy} ${cz}" rpy="0 0 0"/> <!-- This origin is where child link is placed w.r.t parent link -->
+            <limit effort="1000" velocity="1000"/>
+            <dynamics damping="1.0" friction="1.0"/>
         </joint>
         <!-- Define the wheel module link -->
