Commit message: latlon waypoint follower now works

File: sim_ws/src/nav2_gps_waypoint_follower_demo/urdf/gazebo.xacro (robot description, xacro)
@@ -53,6 +53,6 @@
     <material>Gazebo/Black</material>
   </gazebo> -->
-  <gazebo reference="chassis_link">
-    <material>Gazebo/Black</material>
+  <gazebo reference="chassis">
+    <material>Gazebo/Grey</material>
   </gazebo>
   <gazebo reference="base_scan">
