Commit message: reduced mass on components

File: sim_ws/src/nav2_gps_waypoint_follower_demo/urdf/acorn.urdf.xacro (robot description, xacro)
@@ -10,5 +10,5 @@
     <!-- <xacro:arg name="is_simulation" default="true" /> -->
     <!-- Chassis dimensions -->
-    <xacro:property name="chassis_mass" value="30.0"/> <!-- kilograms -->
+    <xacro:property name="chassis_mass" value="1.0"/> <!-- kilograms -->
     <xacro:property name="chassis_length" value="3"/> <!-- meters -->
     <xacro:property name="chassis_width" value="1.5"/>
@@ -21,5 +21,5 @@
     <xacro:property name="module_height" value="0.8"/>
     <!-- Wheel dimensions -->
-    <xacro:property name="wheel_mass" value="1.0"/> <!-- kilograms -->
+    <xacro:property name="wheel_mass" value="0.1"/> <!-- kilograms -->
     <xacro:property name="wheel_radius" value="0.3"/> <!-- meters -->
     <xacro:property name="wheel_width" value="0.1"/>

File: sim_ws/src/nav2_gps_waypoint_follower_demo/urdf/gazebo.xacro (robot description, xacro)
@@ -2,15 +2,5 @@
 <robot xmlns:xacro="http://www.ros.org/wiki/xacro">
   <!-- Gazebo references for moving parts -->
-  <gazebo reference="chassis_link">
-    <kp>10000.0</kp>
-    <kd>10.0</kd>
-    <mu1>1.5</mu1>
-    <mu2>1.5</mu2>
-    <fdir1>0.1 0 0</fdir1>
-    <maxVel>10.0</maxVel>
-    <minDepth>0.0005</minDepth>
-    <material>Gazebo/Black</material>
-  </gazebo>
-  <gazebo reference="wheel_module_front_left">
+  <!-- <gazebo reference="wheel_module_front_left">
     <kp>10000.0</kp>
     <kd>10.0</kd>
@@ -51,41 +41,41 @@
     <minDepth>0.0005</minDepth>
     <material>Gazebo/Black</material>
-  </gazebo>
+  </gazebo> -->
   <gazebo reference="wheel_front_left">
     <kp>100000.0</kp>
     <kd>50.0</kd>
     <gravity>1</gravity>
-    <mu1>100</mu1>
-    <mu2>100</mu2>
+    <mu1>100000</mu1>
+    <mu2>100000</mu2>
+    <minDepth>0.001</minDepth>
+    <implicitSpringDamper>1</implicitSpringDamper>
+    <material>Gazebo/Grey</material>
+  </gazebo>
+  <gazebo reference="wheel_front_right">
+    <kp>100000.0</kp>
+    <kd>50.0</kd>
+    <gravity>1</gravity>
+    <mu1>100000</mu1>
+    <mu2>100000</mu2>
     <minDepth>0.00</minDepth>
     <implicitSpringDamper>1</implicitSpringDamper>
     <material>Gazebo/Grey</material>
   </gazebo>
-  <gazebo reference="wheel_front_right">
-    <kp>100000.0</kp>
-    <kd>50.0</kd>
-    <gravity>1</gravity>
-    <mu1>100</mu1>
-    <mu2>100</mu2>
+  <gazebo reference="wheel_rear_left">
+    <kp>100000.0</kp>
+    <kd>50.0</kd>
+    <gravity>1</gravity>
+    <mu1>100000</mu1>
+    <mu2>100000</mu2>
     <minDepth>0.00</minDepth>
     <implicitSpringDamper>1</implicitSpringDamper>
     <material>Gazebo/Grey</material>
   </gazebo>
-  <gazebo reference="wheel_rear_left">
-    <kp>100000.0</kp>
-    <kd>50.0</kd>
-    <gravity>1</gravity>
-    <mu1>100</mu1>
-    <mu2>100</mu2>
-    <minDepth>0.00</minDepth>
-    <implicitSpringDamper>1</implicitSpringDamper>
-    <material>Gazebo/Grey</material>
-  </gazebo>
   <gazebo reference="wheel_rear_right">
     <kp>100000.0</kp>
     <kd>50.0</kd>
     <gravity>1</gravity>
-    <mu1>100</mu1>
-    <mu2>100</mu2>
+    <mu1>100000</mu1>
+    <mu2>100000</mu2>
     <minDepth>0.00</minDepth>
     <implicitSpringDamper>1</implicitSpringDamper>
@@ -219,6 +209,6 @@
       <joint_name>wheel_front_left_joint</joint_name>
       <joint_name>wheel_front_right_joint</joint_name>
-      <joint_name>wheel_rear_left_joint</joint_name>
-      <joint_name>wheel_rear_right_joint</joint_name>
+      <!-- <joint_name>wheel_rear_left_joint</joint_name> -->
+      <!-- <joint_name>wheel_rear_right_joint</joint_name> -->
     </plugin>
     <!-- Skid Steer Drive Plugin -->
@@ -228,14 +218,14 @@
         <remapping>/tf:=tf</remapping>
       </ros>
-      <num_wheel_pairs>2</num_wheel_pairs>
+      <!-- <num_wheel_pairs>2</num_wheel_pairs> -->
       <update_rate>30</update_rate>
       <left_joint>wheel_front_left_joint</left_joint>
       <right_joint>wheel_front_right_joint</right_joint>
-      <left_joint>wheel_rear_left_joint</left_joint>
-      <right_joint>wheel_rear_right_joint</right_joint>
-      <wheel_separation>1.2</wheel_separation>
+      <!-- <left_joint>wheel_rear_left_joint</left_joint> -->
+      <!-- <right_joint>wheel_rear_right_joint</right_joint> -->
+      <!-- <wheel_separation>1.2</wheel_separation> -->
       <wheel_separation>1.2</wheel_separation>
       <wheel_diameter>0.3</wheel_diameter>
-      <wheel_diameter>0.3</wheel_diameter>
+      <!-- <wheel_diameter>0.3</wheel_diameter> -->
       <publish_odom>true</publish_odom>
       <publish_odom_tf>false</publish_odom_tf>

File: sim_ws/src/nav2_gps_waypoint_follower_demo/urdf/wheel_module_macro.xacro (robot description, xacro)
@@ -45,5 +45,5 @@
             </collision>
             <!-- !Hardcoded mass -->
-            <xacro:inertial_box mass="2.0" x="${module_width_x}" y="${module_width_y}" z="${module_len}">
+            <xacro:inertial_box mass="0.1" x="${module_width_x}" y="${module_width_y}" z="${module_len}">
                 <origin xyz="0 0 0" rpy="0 0 0"/>
             </xacro:inertial_box>

Commit message: robot does not turn

File: sim_ws/src/nav2_gps_waypoint_follower_demo/urdf/acorn.urdf.xacro (robot description, xacro)
@@ -1,4 +1,4 @@
 <?xml version="1.0"?>
-<robot xmlns:xacro="http://www.ros.org/wiki/xacro" name="acron">
+<robot xmlns:xacro="http://www.ros.org/wiki/xacro" name="acorn">
     <!-- <xacro:include filename="robot_core.xacro" /> -->
     <!-- REFER TO IMAGES FOLDER FOR VISUAL REPRESENTATION OF THE ROBOT -->
@@ -10,5 +10,5 @@
     <!-- <xacro:arg name="is_simulation" default="true" /> -->
     <!-- Chassis dimensions -->
-    <xacro:property name="chassis_mass" value="1.0"/> <!-- kilograms -->
+    <xacro:property name="chassis_mass" value="30.0"/> <!-- kilograms -->
     <xacro:property name="chassis_length" value="3"/> <!-- meters -->
     <xacro:property name="chassis_width" value="1.5"/>
@@ -21,5 +21,5 @@
     <xacro:property name="module_height" value="0.8"/>
     <!-- Wheel dimensions -->
-    <xacro:property name="wheel_mass" value="0.1"/> <!-- kilograms -->
+    <xacro:property name="wheel_mass" value="5.0"/> <!-- kilograms -->
     <xacro:property name="wheel_radius" value="0.3"/> <!-- meters -->
     <xacro:property name="wheel_width" value="0.1"/>

File: sim_ws/src/nav2_gps_waypoint_follower_demo/urdf/gazebo.xacro (robot description, xacro)
@@ -1,4 +1,5 @@
 <?xml version="1.0"?>
-<robot xmlns:xacro="http://www.ros.org/wiki/xacro">
+<!-- <robot xmlns:xacro="http://www.ros.org/wiki/xacro"> -->
+<robot>
   <!-- Gazebo references for moving parts -->
   <!-- <gazebo reference="wheel_module_front_left">
@@ -42,5 +43,5 @@
     <material>Gazebo/Black</material>
   </gazebo> -->
-  <gazebo reference="wheel_front_left">
+  <!-- <gazebo reference="chassis_link">
     <kp>100000.0</kp>
     <kd>50.0</kd>
@@ -50,34 +51,49 @@
     <minDepth>0.001</minDepth>
     <implicitSpringDamper>1</implicitSpringDamper>
+    <material>Gazebo/Black</material>
+  </gazebo> -->
+  <gazebo reference="chassis_link">
+    <mul1>0.2</mul1>
+    <mul2>0.2</mul2>
+    <material>Gazebo/Black</material>
+  </gazebo>
+  <gazebo reference="wheel_module_front_left">
+    <mul1>0.2</mul1>
+    <mul2>0.2</mul2>
+    <material>Gazebo/Grey</material>
+  </gazebo>
+  <gazebo reference="wheel_module_front_right">
+    <mul1>0.2</mul1>
+    <mul2>0.2</mul2>
+    <material>Gazebo/Grey</material>
+  </gazebo>
+  <gazebo reference="wheel_module_rear_left">
+    <mul1>0.2</mul1>
+    <mul2>0.2</mul2>
+    <material>Gazebo/Grey</material>
+  </gazebo>
+  <gazebo reference="wheel_module_rear_right">
+    <mul1>0.2</mul1>
+    <mul2>0.2</mul2>
+    <material>Gazebo/Grey</material>
+  </gazebo>
+  <gazebo reference="wheel_front_left">
+    <mul1>0.2</mul1>
+    <mul2>0.2</mul2>
     <material>Gazebo/Grey</material>
   </gazebo>
   <gazebo reference="wheel_front_right">
-    <kp>100000.0</kp>
-    <kd>50.0</kd>
-    <gravity>1</gravity>
-    <mu1>100000</mu1>
-    <mu2>100000</mu2>
-    <minDepth>0.00</minDepth>
-    <implicitSpringDamper>1</implicitSpringDamper>
+    <mul1>0.2</mul1>
+    <mul2>0.2</mul2>
     <material>Gazebo/Grey</material>
   </gazebo>
   <gazebo reference="wheel_rear_left">
-    <kp>100000.0</kp>
-    <kd>50.0</kd>
-    <gravity>1</gravity>
-    <mu1>100000</mu1>
-    <mu2>100000</mu2>
-    <minDepth>0.00</minDepth>
-    <implicitSpringDamper>1</implicitSpringDamper>
+    <mul1>0.2</mul1>
+    <mul2>0.2</mul2>
     <material>Gazebo/Grey</material>
   </gazebo>
   <gazebo reference="wheel_rear_right">
-    <kp>100000.0</kp>
-    <kd>50.0</kd>
-    <gravity>1</gravity>
-    <mu1>100000</mu1>
-    <mu2>100000</mu2>
-    <minDepth>0.00</minDepth>
-    <implicitSpringDamper>1</implicitSpringDamper>
+    <mul1>0.2</mul1>
+    <mul2>0.2</mul2>
     <material>Gazebo/Grey</material>
   </gazebo>
@@ -207,8 +223,9 @@
           <remapping>~/out:=joint_states</remapping>
       </ros>
+      <update_rate>30</update_rate>
       <joint_name>wheel_front_left_joint</joint_name>
       <joint_name>wheel_front_right_joint</joint_name>
-      <!-- <joint_name>wheel_rear_left_joint</joint_name> -->
-      <!-- <joint_name>wheel_rear_right_joint</joint_name> -->
+      <joint_name>wheel_rear_left_joint</joint_name>
+      <joint_name>wheel_rear_right_joint</joint_name>
     </plugin>
     <!-- Skid Steer Drive Plugin -->
@@ -218,14 +235,17 @@
         <remapping>/tf:=tf</remapping>
       </ros>
-      <!-- <num_wheel_pairs>2</num_wheel_pairs> -->
+      <num_wheel_pairs>2</num_wheel_pairs>
       <update_rate>30</update_rate>
+      <!-- Wheel pair 1 -->
       <left_joint>wheel_front_left_joint</left_joint>
       <right_joint>wheel_front_right_joint</right_joint>
-      <!-- <left_joint>wheel_rear_left_joint</left_joint> -->
-      <!-- <right_joint>wheel_rear_right_joint</right_joint> -->
-      <!-- <wheel_separation>1.2</wheel_separation> -->
+      <!-- Wheel pair 2 -->
+      <left_joint>wheel_rear_left_joint</left_joint>
+      <right_joint>wheel_rear_right_joint</right_joint>
+      <!-- Kinematics -->
+      <wheel_separation>1.2</wheel_separation>
       <wheel_separation>1.2</wheel_separation>
       <wheel_diameter>0.3</wheel_diameter>
-      <!-- <wheel_diameter>0.3</wheel_diameter> -->
+      <wheel_diameter>0.3</wheel_diameter>
       <publish_odom>true</publish_odom>
       <publish_odom_tf>false</publish_odom_tf>
@@ -234,5 +254,5 @@
       <odometry_topic>odom</odometry_topic>
       <odometry_frame>odom</odometry_frame>
-      <robot_base_frame>base_link</robot_base_frame>
+      <robot_base_frame>base_footprint</robot_base_frame>
       <max_wheel_torque>1000</max_wheel_torque>
       <max_acceleration>20.0</max_acceleration>

File: sim_ws/src/nav2_gps_waypoint_follower_demo/urdf/wheel_module_macro.xacro (robot description, xacro)
@@ -3,4 +3,24 @@
     <include filename="color_macro.xacro"/>
     <include filename="inertia_macro.xacro"/>
+    <!-- Wheel dimensions -->
+    <xacro:property name="wheel_link_radius" value="0.15"/>
+    <xacro:property name="wheel_link_length" value="0.1"/>
+    <!-- Material Density -->
+    <xacro:property name="wheel_density" value="2710.0"/>
+    <!-- Pi Constant -->
+    <xacro:property name="pi_const" value="3.141592265"/>
+    <!-- Robot body and wheel mass -->
+    <xacro:property name="wheel_mass" value="${wheel_density*pi_const*wheel_link_radius*wheel_link_radius*wheel_link_length}"/>
+    <!-- Moments of inertial of the wheel -->
+    <xacro:property name="Iz_wheel" value="${0.5*wheel_mass*wheel_link_radius*wheel_link_radius}"/>
+    <xacro:property name="I_wheel" value="${(1.0/12.0)*wheel_mass*(3*wheel_link_radius*wheel_link_radius+wheel_link_length*wheel_link_length)}"/>
+    <!-- macros -->
+    <xacro:macro name="inertia_wheel">
+        <inertial>
+            <origin rpy="0 0 0" xyz="0 0 0"/>
+            <mass value="${wheel_mass}"/>
+            <inertia ixx="${I_wheel}" ixy="0.0" ixz="0.0" iyy="${I_wheel}" iyz="0" izz="${Iz_wheel}"/>
+        </inertial>
+    </xacro:macro>
     <!--
         A macro to create a wheel module (including links and joints)
@@ -52,5 +72,5 @@
         <xacro:if value="${side == 'left'}">
             <xacro:property name="wheel_position_y" value="${width}"/>
-            <xacro:property name="wheel_pitch" value="-${PI/2}"/>
+            <xacro:property name="wheel_pitch" value="${PI/2}"/>
         </xacro:if>
         <xacro:if value="${side == 'right'}">
@@ -61,9 +81,12 @@
             <parent link="wheel_module_${parent_name}"/>
             <child link="wheel_${parent_name}"/>
-            <origin xyz="0 ${wheel_position_y} ${-module_len/2.0}" rpy="${wheel_pitch} 0 0"/>
-            <axis xyz="0 0 1"/>
+            <origin xyz="0 ${wheel_position_y} ${-module_len/2.0}" rpy="0 0 0"/>
+            <axis xyz="0 1 0"/>
+            <limit effort="1000" velocity="1000"/>
+            <dynamics damping="1.0" friction="1.0"/>
         </joint>
         <link name="wheel_${parent_name}">
             <visual>
+                <origin rpy="${wheel_pitch} 0 0" xyz="0 0 0"/>
                 <geometry>
                     <cylinder radius="${radius}" length="${width}"/>
@@ -72,11 +95,13 @@
             </visual>
             <collision>
+                <origin rpy="${wheel_pitch} 0 0" xyz="0 0 0"/>
                 <geometry>
                     <cylinder radius="${radius}" length="${width}"/>
                 </geometry>
             </collision>
-            <xacro:inertial_cylinder mass="${mass}" length="${width}" radius="${radius}">
+            <!-- <xacro:inertial_cylinder mass="${mass}" length="${width}" radius="${radius}">
                 <origin xyz="0 0 0" rpy="0 0 0"/>
-            </xacro:inertial_cylinder>
+            </xacro:inertial_cylinder> -->
+            <xacro:inertia_wheel />
         </link>
     </xacro:macro>

Commit message: added lidar

File: sim_ws/src/nav2_gps_waypoint_follower_demo/urdf/acorn.urdf.xacro (robot description, xacro)
@@ -107,5 +107,15 @@
         <origin xyz="0 0 0" rpy="0 0 0"/>
     </joint>
-    <link name="gps_link"/>
+    <link name="gps_link">
+        <inertial>
+            <mass>0.001</mass>
+            <ixx>0.001</ixx>
+            <ixy>0.000</ixy>
+            <ixz>0.000</ixz>
+            <iyy>0.001</iyy>
+            <iyz>0.000</iyz>
+            <izz>0.001</izz>
+        </inertial>
+    </link>
     <!-- 2D Lidar placed in front center 20cm below chassis-->
     <joint name="scan_joint" type="fixed">
@@ -117,4 +127,7 @@
         <visual>
         <origin xyz="0 0 0" rpy="0 0 0"/>
+        <geometry>
+            <mesh filename="package://turtlebot3_gazebo/models/turtlebot3_common/meshes/lds.dae" scale="0.001 0.001 0.001"/>
+        </geometry>
         <material name="dark"/>
         </visual>

File: sim_ws/src/nav2_gps_waypoint_follower_demo/urdf/gazebo.xacro (robot description, xacro)
@@ -54,4 +54,7 @@
   </gazebo> -->
   <gazebo reference="chassis_link">
+    <material>Gazebo/Black</material>
+  </gazebo>
+  <gazebo reference="base_scan">
     <material>Gazebo/Black</material>
   </gazebo>
@@ -139,5 +142,5 @@
         </noise>
       </ray>
-      <plugin filename="libgazebo_ros_ray_sensor.so" name="lidar_1">
+      <plugin name="turtlebot3_laserscan" filename="libgazebo_ros_ray_sensor.so">
         <ros>
           <argument>~/out:=scan</argument>

Commit message: acorn now works in nav2 outdoor world

File: sim_ws/src/nav2_gps_waypoint_follower_demo/urdf/acorn.urdf.xacro (robot description, xacro)
@@ -1,4 +1,4 @@
 <?xml version="1.0"?>
-<robot xmlns:xacro="http://www.ros.org/wiki/xacro" name="robot">
+<robot xmlns:xacro="http://www.ros.org/wiki/xacro" name="acorn">
     <!-- <xacro:include filename="robot_core.xacro" /> -->
     <!-- REFER TO IMAGES FOLDER FOR VISUAL REPRESENTATION OF THE ROBOT -->
@@ -11,15 +11,15 @@
     <!-- Chassis dimensions -->
     <xacro:property name="chassis_mass" value="30.0"/> <!-- kilograms -->
-    <xacro:property name="chassis_length" value="3"/> <!-- meters -->
-    <xacro:property name="chassis_width" value="1.5"/>
+    <xacro:property name="chassis_length" value="2"/> <!-- meters -->
+    <xacro:property name="chassis_width" value="2"/>
     <xacro:property name="chassis_height" value="0.3"/>
     <!-- Wheel Module dimensions -->
-    <xacro:property name="base_to_module_x" value="1.2"/> <!-- meters -->
-    <xacro:property name="base_to_module_y" value="0.6"/>
+    <xacro:property name="base_to_module_x" value="0.8"/> <!-- meters -->
+    <xacro:property name="base_to_module_y" value="0.8"/>
     <xacro:property name="module_width_x" value="0.2"/>
     <xacro:property name="module_width_y" value="0.15"/>
     <xacro:property name="module_height" value="0.8"/>
     <!-- Wheel dimensions -->
-    <xacro:property name="wheel_mass" value="1.0"/> <!-- kilograms -->
+    <xacro:property name="wheel_mass" value="5.0"/> <!-- kilograms -->
     <xacro:property name="wheel_radius" value="0.3"/> <!-- meters -->
     <xacro:property name="wheel_width" value="0.1"/>
@@ -107,5 +107,15 @@
         <origin xyz="0 0 0" rpy="0 0 0"/>
     </joint>
-    <link name="gps_link"/>
+    <link name="gps_link">
+        <inertial>
+            <mass>0.001</mass>
+            <ixx>0.001</ixx>
+            <ixy>0.000</ixy>
+            <ixz>0.000</ixz>
+            <iyy>0.001</iyy>
+            <iyz>0.000</iyz>
+            <izz>0.001</izz>
+        </inertial>
+    </link>
     <!-- 2D Lidar placed in front center 20cm below chassis-->
     <joint name="scan_joint" type="fixed">
@@ -136,3 +146,5 @@
         </inertial>
     </link>
+    <!-- Include gazebo macros for sim -->
+    <xacro:include filename="gazebo.xacro" />
 </robot>

File: sim_ws/src/nav2_gps_waypoint_follower_demo/urdf/wheel_module_macro.xacro (robot description, xacro)
@@ -3,4 +3,24 @@
     <include filename="color_macro.xacro"/>
     <include filename="inertia_macro.xacro"/>
+    <!-- Wheel dimensions -->
+    <xacro:property name="wheel_link_radius" value="0.15"/>
+    <xacro:property name="wheel_link_length" value="0.1"/>
+    <!-- Material Density -->
+    <xacro:property name="wheel_density" value="2710.0"/>
+    <!-- Pi Constant -->
+    <xacro:property name="pi_const" value="3.141592265"/>
+    <!-- Robot body and wheel mass -->
+    <xacro:property name="wheel_mass" value="${wheel_density*pi_const*wheel_link_radius*wheel_link_radius*wheel_link_length}"/>
+    <!-- Moments of inertial of the wheel -->
+    <xacro:property name="Iz_wheel" value="${0.5*wheel_mass*wheel_link_radius*wheel_link_radius}"/>
+    <xacro:property name="I_wheel" value="${(1.0/12.0)*wheel_mass*(3*wheel_link_radius*wheel_link_radius+wheel_link_length*wheel_link_length)}"/>
+    <!-- macros -->
+    <xacro:macro name="inertia_wheel">
+        <inertial>
+            <origin rpy="0 0 0" xyz="0 0 0"/>
+            <mass value="${wheel_mass}"/>
+            <inertia ixx="${I_wheel}" ixy="0.0" ixz="0.0" iyy="${I_wheel}" iyz="0" izz="${Iz_wheel}"/>
+        </inertial>
+    </xacro:macro>
     <!--
         A macro to create a wheel module (including links and joints)
@@ -26,4 +46,6 @@
             <child link="wheel_module_${parent_name}"/>
             <origin xyz="${cx} ${cy} ${cz}" rpy="0 0 0"/> <!-- This origin is where child link is placed w.r.t parent link -->
+            <!-- <limit effort="1000" velocity="1000"/> -->
+            <!-- <dynamics damping="1.0" friction="1.0"/> -->
         </joint>
         <!-- Define the wheel module link -->
@@ -43,5 +65,5 @@
             </collision>
             <!-- !Hardcoded mass -->
-            <xacro:inertial_box mass="2.0" x="${module_width_x}" y="${module_width_y}" z="${module_len}">
+            <xacro:inertial_box mass="0.1" x="${module_width_x}" y="${module_width_y}" z="${module_len}">
                 <origin xyz="0 0 0" rpy="0 0 0"/>
             </xacro:inertial_box>
@@ -50,5 +72,5 @@
         <xacro:if value="${side == 'left'}">
             <xacro:property name="wheel_position_y" value="${width}"/>
-            <xacro:property name="wheel_pitch" value="-${PI/2}"/>
+            <xacro:property name="wheel_pitch" value="${PI/2}"/>
         </xacro:if>
         <xacro:if value="${side == 'right'}">
@@ -59,9 +81,12 @@
             <parent link="wheel_module_${parent_name}"/>
             <child link="wheel_${parent_name}"/>
-            <origin xyz="0 ${wheel_position_y} ${-module_len/2.0}" rpy="${wheel_pitch} 0 0"/>
-            <axis xyz="0 0 1"/>
+            <origin xyz="0 ${wheel_position_y} ${-module_len/2.0}" rpy="0 0 0"/>
+            <axis xyz="0 1 0"/>
+            <limit effort="2000" velocity="2000"/>
+            <dynamics damping="1.0" friction="0.5"/>
         </joint>
         <link name="wheel_${parent_name}">
             <visual>
+                <origin rpy="${wheel_pitch} 0 0" xyz="0 0 0"/>
                 <geometry>
                     <cylinder radius="${radius}" length="${width}"/>
@@ -70,11 +95,13 @@
             </visual>
             <collision>
+                <origin rpy="${wheel_pitch} 0 0" xyz="0 0 0"/>
                 <geometry>
                     <cylinder radius="${radius}" length="${width}"/>
                 </geometry>
             </collision>
-            <xacro:inertial_cylinder mass="${mass}" length="${width}" radius="${radius}">
+            <!-- <xacro:inertial_cylinder mass="${mass}" length="${width}" radius="${radius}">
                 <origin xyz="0 0 0" rpy="0 0 0"/>
-            </xacro:inertial_cylinder>
+            </xacro:inertial_cylinder> -->
+            <xacro:inertia_wheel />
         </link>
     </xacro:macro>
