Commit message: added 4 wheel steering control to urdf. Need to integrate nav2

File: sim_ws/src/nav2_gps_waypoint_follower_demo/urdf/acorn.urdf.xacro (robot description, xacro)
@@ -146,4 +146,34 @@
         </inertial>
     </link>
+    <!-- CONTROLLERS -->
+    <xacro:macro name="steering_module_controller" params="name">
+        <joint name="wheel_module_${parent_name}_joint">
+            <command_interface name="position">
+                <param name="min">-${2 * PI}</param>
+                <param name="max">${2 * PI}</param>
+            </command_interface>
+            <state_interface name="position"/>
+            <state_interface name="velocity"/>
+            <state_interface name="acceleration"/>
+        </joint>
+        <joint name="wheel_${name}_joint">
+            <command_interface name="velocity">
+                <param name="min">-1</param>
+                <param name="max">1</param>
+            </command_interface>
+            <state_interface name="position"/>
+            <state_interface name="velocity"/>
+            <state_interface name="acceleration"/>
+        </joint>
+    </xacro:macro>
+    <ros2_control name="ZingerJointControl" type="system">
+        <hardware>
+            <plugin>ign_ros2_control/IgnitionSystem</plugin>
+        </hardware>
+        <xacro:steering_module_controller name="front_left" />
+        <xacro:steering_module_controller name="rear_left" />
+        <xacro:steering_module_controller name="rear_right" />
+        <xacro:steering_module_controller name="front_right" />
+    </ros2_control>
     <!-- Include gazebo macros for sim -->
     <xacro:include filename="gazebo.xacro" />

File: sim_ws/src/nav2_gps_waypoint_follower_demo/urdf/gazebo.xacro (robot description, xacro)
@@ -3,54 +3,4 @@
 <robot>
   <!-- Gazebo references for moving parts -->
-  <!-- <gazebo reference="wheel_module_front_left">
-    <kp>10000.0</kp>
-    <kd>10.0</kd>
-    <mu1>1.5</mu1>
-    <mu2>1.5</mu2>
-    <fdir1>0.1 0 0</fdir1>
-    <maxVel>10.0</maxVel>
-    <minDepth>0.0005</minDepth>
-    <material>Gazebo/Black</material>
-  </gazebo>
-  <gazebo reference="wheel_module_front_right">
-    <kp>10000.0</kp>
-    <kd>10.0</kd>
-    <mu1>1.5</mu1>
-    <mu2>1.5</mu2>
-    <fdir1>0.1 0 0</fdir1>
-    <maxVel>10.0</maxVel>
-    <minDepth>0.0005</minDepth>
-    <material>Gazebo/Black</material>
-  </gazebo>
-  <gazebo reference="wheel_module_rear_left">
-    <kp>10000.0</kp>
-    <kd>10.0</kd>
-    <mu1>1.5</mu1>
-    <mu2>1.5</mu2>
-    <fdir1>0.1 0 0</fdir1>
-    <maxVel>10.0</maxVel>
-    <minDepth>0.0005</minDepth>
-    <material>Gazebo/Black</material>
-  </gazebo>
-  <gazebo reference="wheel_module_rear_right">
-    <kp>10000.0</kp>
-    <kd>10.0</kd>
-    <mu1>1.5</mu1>
-    <mu2>1.5</mu2>
-    <fdir1>0.1 0 0</fdir1>
-    <maxVel>10.0</maxVel>
-    <minDepth>0.0005</minDepth>
-    <material>Gazebo/Black</material>
-  </gazebo> -->
-  <!-- <gazebo reference="chassis_link">
-    <kp>100000.0</kp>
-    <kd>50.0</kd>
-    <gravity>1</gravity>
-    <mu1>100000</mu1>
-    <mu2>100000</mu2>
-    <minDepth>0.001</minDepth>
-    <implicitSpringDamper>1</implicitSpringDamper>
-    <material>Gazebo/Black</material>
-  </gazebo> -->
   <gazebo reference="chassis">
     <material>Gazebo/Grey</material>
@@ -60,57 +10,53 @@
   </gazebo>
   <gazebo reference="wheel_module_front_left">
-    <mul1>1.0</mul1>
-    <mul2>1.0</mul2>
-    <slip1>0.1</slip1>
-    <slip2>0.1</slip2>
     <material>Gazebo/Grey</material>
   </gazebo>
   <gazebo reference="wheel_module_front_right">
-    <mul1>1.0</mul1>
-    <mul2>1.0</mul2>
-    <slip1>0.1</slip1>
-    <slip2>0.1</slip2>
     <material>Gazebo/Grey</material>
   </gazebo>
   <gazebo reference="wheel_module_rear_left">
-    <mul1>1.0</mul1>
-    <mul2>1.0</mul2>
-    <slip1>0.1</slip1>
-    <slip2>0.1</slip2>
     <material>Gazebo/Grey</material>
   </gazebo>
   <gazebo reference="wheel_module_rear_right">
-    <mul1>1.0</mul1>
-    <mul2>1.0</mul2>
-    <slip1>0.1</slip1>
-    <slip2>0.1</slip2>
     <material>Gazebo/Grey</material>
   </gazebo>
   <gazebo reference="wheel_front_left">
-    <mul1>1.0</mul1>
-    <mul2>1.0</mul2>
-    <slip1>0.1</slip1>
-    <slip2>0.1</slip2>
+    <mu1>0.9</mu1>
+    <mu2>0.9</mu2>
+    <kp>500000.0</kp>
+    <kd>10.0</kd>
+    <minDepth>0.001</minDepth>
+    <maxVel>0.1</maxVel>
+    <fdir1>1 0 0</fdir1>
     <material>Gazebo/Grey</material>
   </gazebo>
   <gazebo reference="wheel_front_right">
-    <mul1>1.0</mul1>
-    <mul2>1.0</mul2>
-    <slip1>0.1</slip1>
-    <slip2>0.1</slip2>
+    <mu1>0.9</mu1>
+    <mu2>0.9</mu2>
+    <kp>500000.0</kp>
+    <kd>10.0</kd>
+    <minDepth>0.001</minDepth>
+    <maxVel>0.1</maxVel>
+    <fdir1>1 0 0</fdir1>
     <material>Gazebo/Grey</material>
   </gazebo>
   <gazebo reference="wheel_rear_left">
-    <mul1>1.0</mul1>
-    <mul2>1.0</mul2>
-    <slip1>0.1</slip1>
-    <slip2>0.1</slip2>
+    <mu1>0.9</mu1>
+    <mu2>0.9</mu2>
+    <kp>500000.0</kp>
+    <kd>10.0</kd>
+    <minDepth>0.001</minDepth>
+    <maxVel>0.1</maxVel>
+    <fdir1>1 0 0</fdir1>
     <material>Gazebo/Grey</material>
   </gazebo>
   <gazebo reference="wheel_rear_right">
-    <mul1>1.0</mul1>
-    <mul2>1.0</mul2>
-    <slip1>0.1</slip1>
-    <slip2>0.1</slip2>
+    <mu1>0.9</mu1>
+    <mu2>0.9</mu2>
+    <kp>500000.0</kp>
+    <kd>10.0</kd>
+    <minDepth>0.001</minDepth>
+    <maxVel>0.1</maxVel>
+    <fdir1>1 0 0</fdir1>
     <material>Gazebo/Grey</material>
   </gazebo>
@@ -233,46 +179,26 @@
     </sensor>
   </gazebo>
-  <!-- Add the skid steering plugin to the robot model -->
+  <!-- Add the 4 wheel steering plugin to the robot model -->
   <gazebo>
-    <!-- Specify joint state publisher here or launch node separately -->
-    <plugin name="joint_states" filename="libgazebo_ros_joint_state_publisher.so">
-      <ros>
-          <remapping>~/out:=joint_states</remapping>
-      </ros>
-      <update_rate>30</update_rate>
-      <joint_name>wheel_front_left_joint</joint_name>
-      <joint_name>wheel_front_right_joint</joint_name>
-      <joint_name>wheel_rear_left_joint</joint_name>
-      <joint_name>wheel_rear_right_joint</joint_name>
-    </plugin>
-    <!-- Skid Steer Drive Plugin -->
-    <!-- NOTE: Skid steer plugin merged with diff drive in ros2 -->
-    <plugin name='diff_drive' filename='libgazebo_ros_diff_drive.so'>
-      <ros>
-        <remapping>/tf:=tf</remapping>
-      </ros>
-      <num_wheel_pairs>2</num_wheel_pairs>
-      <update_rate>30</update_rate>
-      <!-- Wheel pair 1 -->
-      <left_joint>wheel_front_left_joint</left_joint>
-      <right_joint>wheel_front_right_joint</right_joint>
-      <!-- Wheel pair 2 -->
-      <left_joint>wheel_rear_left_joint</left_joint>
-      <right_joint>wheel_rear_right_joint</right_joint>
-      <!-- Kinematics -->
-      <wheel_separation>2.0</wheel_separation>
-      <wheel_separation>2.0</wheel_separation>
-      <wheel_diameter>0.3</wheel_diameter>
-      <wheel_diameter>0.3</wheel_diameter>
-      <publish_odom>true</publish_odom>
-      <publish_odom_tf>false</publish_odom_tf>
-      <publish_wheel_tf>false</publish_wheel_tf>
-      <command_topic>cmd_vel</command_topic>
-      <odometry_topic>odom</odometry_topic>
-      <odometry_frame>odom</odometry_frame>
-      <robot_base_frame>base_footprint</robot_base_frame>
-      <max_wheel_torque>1000</max_wheel_torque>
-      <max_acceleration>30.0</max_acceleration>
-    </plugin>
+      <plugin
+              filename="ign_ros2_control-system"
+              name="ign_ros2_control::IgnitionROS2ControlPlugin">
+          <parameters>$(find nav2_gps_waypoint_follower_demo)/config/zinger.yaml</parameters>
+      </plugin>
+  </gazebo>
+  <gazebo>
+        <plugin
+              filename="libignition-gazebo-pose-publisher-system.so"
+              name="ignition::gazebo::systems::PosePublisher">
+          <publish_link_pose>true</publish_link_pose>
+          <publish_sensor_pose>true</publish_sensor_pose>
+          <publish_collision_pose>false</publish_collision_pose>
+          <publish_visual_pose>false</publish_visual_pose>
+          <publish_model_pose>true</publish_model_pose>
+          <publish_nested_model_pose>true</publish_nested_model_pose>
+          <use_pose_vector_msg>true</use_pose_vector_msg>
+          <static_publisher>true</static_publisher>
+          <static_update_frequency>-1</static_update_frequency>
+      </plugin>
   </gazebo>
 </robot>

File: sim_ws/src/nav2_gps_waypoint_follower_demo/urdf/wheel_module_macro.xacro (robot description, xacro)
@@ -42,8 +42,9 @@
         Then create a joint to connect the wheel to the wheel module
         -->
-        <joint name="wheel_module_${parent_name}_joint" type="fixed">
+        <joint name="wheel_module_${parent_name}_joint" type="continuous">
             <parent link="${parent_name}"/>
             <child link="wheel_module_${parent_name}"/>
             <origin xyz="${cx} ${cy} ${cz}" rpy="0 0 0"/> <!-- This origin is where child link is placed w.r.t parent link -->
+            <axis xyz="0 0 1"/>
             <!-- <limit effort="1000" velocity="1000"/> -->
             <!-- <dynamics damping="1.0" friction="1.0"/> -->
@@ -100,7 +101,4 @@
                 </geometry>
             </collision>
-            <!-- <xacro:inertial_cylinder mass="${mass}" length="${width}" radius="${radius}">
-                <origin xyz="0 0 0" rpy="0 0 0"/>
-            </xacro:inertial_cylinder> -->
             <xacro:inertia_wheel />
         </link>

Commit message: bug fixes in launch file

File: sim_ws/src/nav2_gps_waypoint_follower_demo/urdf/acorn.urdf.xacro (robot description, xacro)
@@ -148,5 +148,5 @@
     <!-- CONTROLLERS -->
     <xacro:macro name="steering_module_controller" params="name">
-        <joint name="wheel_module_${parent_name}_joint">
+        <joint name="wheel_module_${name}_joint">
             <command_interface name="position">
                 <param name="min">-${2 * PI}</param>
