Commit message: updated launch files

File: sim_ws/src/simulation_launch/description/robot.urdf.xacro (robot description, xacro)
@@ -31,5 +31,5 @@
         <parent link="base_link"/>
         <child link="chassis"/>
-        Place the chassis at half of chassis height above the base link
+        <!-- Place the chassis at half of chassis height above the base link -->
         <origin xyz="0 0 ${chassis_height/2.0}" rpy="0 0 0"/>
     </joint>
@@ -51,4 +51,5 @@
             <origin xyz="0 0 0" rpy="0 0 0"/>
         </xacro:inertial_box>
+    </link>
     <!-- Define joints to connect static links to the base link -->
     <joint name="FL_joint" type="fixed">

File: sim_ws/src/simulation_launch/description/wheel_module_macro.xacro (robot description, xacro)
@@ -1,4 +1,4 @@
 <?xml version="1.0" ?>
-<robot xmlns:xacro="http://www.ros.org/wiki/xacro" >
+<robot xmlns:xacro="http://www.ros.org/wiki/xacro">
     <include filename="color_macro.xacro"/>
     <include filename="inertia_macro.xacro"/>
@@ -25,10 +25,10 @@
             <parent link="${parent_name}"/>
             <child link="wheel_module_${parent_name}"/>
-            <origin xyz="${cx} ${cy} ${cz}" rpy="0 0 0"/> <!--This origin is where child link is placed w.r.t parent link -->
+            <origin xyz="${cx} ${cy} ${cz}" rpy="0 0 0"/> <!-- This origin is where child link is placed w.r.t parent link -->
         </joint>
         <!-- Define the wheel module link -->
         <link name="wheel_module_${parent_name}">
             <visual>
-                <origin xyz="0 0 0"/> <!--This origin is w.r.t the wheel_module_${parent_name} link -->
+                <origin xyz="0 0 0"/> <!-- This origin is w.r.t the wheel_module_${parent_name} link -->
                 <geometry>
                     <box size="${module_width_x} ${module_width_y} ${module_len}"/>
@@ -37,5 +37,5 @@
             </visual>
             <collision>
-                <origin xyz="0 0 0"/> <!--This origin is w.r.t the wheel_module_${parent_name} link -->
+                <origin xyz="0 0 0"/> <!-- This origin is w.r.t the wheel_module_${parent_name} link -->
                 <geometry>
                     <box size="${module_width_x} ${module_width_y} ${module_len}"/>
