Commit message: bug fixes in urdf and launch files and documentation

File: sim_ws/src/simulation_launch/description/wheel_module_macro.xacro (robot description, xacro)
@@ -22,5 +22,5 @@
         Then create a joint to connect the wheel to the wheel module
         -->
-        <joint name="wheel_module_${parent_name}_joint" type="continuous">
+        <joint name="wheel_module_${parent_name}_joint" type="fixed">
             <parent link="${parent_name}"/>
             <child link="wheel_module_${parent_name}"/>
