Commit message: robot now turns and moves

File: sim_ws/src/mobile_robot/model/robot.xacro (robot description, xacro)
@@ -2,6 +2,6 @@
 <robot name="differential_drive_robot" xmlns:xacro="http://www.ros.org/wiki/xacro">
 <!-- Body dimensions -->
-<xacro:property name="body_link_x_dim" value="1"/>
-<xacro:property name="body_link_y_dim" value="0.6"/>
+<xacro:property name="body_link_x_dim" value="2.0"/>
+<xacro:property name="body_link_y_dim" value="2.0"/>
 <xacro:property name="body_link_z_dim" value="0.3"/>
 <!-- Wheel dimensions -->
@@ -10,6 +10,6 @@
 <xacro:property name="wheel_link_z_location" value="-0.1"/>
 <!-- Material Density -->
-<xacro:property name="body_density" value="2710.0"/>
-<xacro:property name="wheel_density" value="2710.0"/>
+<xacro:property name="body_density" value="20.0"/>
+<xacro:property name="wheel_density" value="20.0"/>
 <!-- Pi Constant -->
 <xacro:property name="pi_const" value="3.141592265"/>

File: sim_ws/src/nav2_gps_waypoint_follower_demo/urdf/acorn.urdf.xacro (robot description, xacro)
@@ -11,10 +11,10 @@
     <!-- Chassis dimensions -->
     <xacro:property name="chassis_mass" value="30.0"/> <!-- kilograms -->
-    <xacro:property name="chassis_length" value="3"/> <!-- meters -->
-    <xacro:property name="chassis_width" value="1.5"/>
+    <xacro:property name="chassis_length" value="2"/> <!-- meters -->
+    <xacro:property name="chassis_width" value="2"/>
     <xacro:property name="chassis_height" value="0.3"/>
     <!-- Wheel Module dimensions -->
-    <xacro:property name="base_to_module_x" value="1.2"/> <!-- meters -->
-    <xacro:property name="base_to_module_y" value="0.6"/>
+    <xacro:property name="base_to_module_x" value="0.8"/> <!-- meters -->
+    <xacro:property name="base_to_module_y" value="0.8"/>
     <xacro:property name="module_width_x" value="0.2"/>
     <xacro:property name="module_width_y" value="0.15"/>

File: sim_ws/src/nav2_gps_waypoint_follower_demo/urdf/gazebo.xacro (robot description, xacro)
@@ -54,46 +54,60 @@
   </gazebo> -->
   <gazebo reference="chassis_link">
-    <mul1>0.2</mul1>
-    <mul2>0.2</mul2>
     <material>Gazebo/Black</material>
   </gazebo>
   <gazebo reference="wheel_module_front_left">
-    <mul1>0.2</mul1>
-    <mul2>0.2</mul2>
+    <mul1>1.0</mul1>
+    <mul2>1.0</mul2>
+    <slip1>0.1</slip1>
+    <slip2>0.1</slip2>
     <material>Gazebo/Grey</material>
   </gazebo>
   <gazebo reference="wheel_module_front_right">
-    <mul1>0.2</mul1>
-    <mul2>0.2</mul2>
+    <mul1>1.0</mul1>
+    <mul2>1.0</mul2>
+    <slip1>0.1</slip1>
+    <slip2>0.1</slip2>
     <material>Gazebo/Grey</material>
   </gazebo>
   <gazebo reference="wheel_module_rear_left">
-    <mul1>0.2</mul1>
-    <mul2>0.2</mul2>
+    <mul1>1.0</mul1>
+    <mul2>1.0</mul2>
+    <slip1>0.1</slip1>
+    <slip2>0.1</slip2>
     <material>Gazebo/Grey</material>
   </gazebo>
   <gazebo reference="wheel_module_rear_right">
-    <mul1>0.2</mul1>
-    <mul2>0.2</mul2>
+    <mul1>1.0</mul1>
+    <mul2>1.0</mul2>
+    <slip1>0.1</slip1>
+    <slip2>0.1</slip2>
     <material>Gazebo/Grey</material>
   </gazebo>
   <gazebo reference="wheel_front_left">
-    <mul1>0.2</mul1>
-    <mul2>0.2</mul2>
+    <mul1>1.0</mul1>
+    <mul2>1.0</mul2>
+    <slip1>0.1</slip1>
+    <slip2>0.1</slip2>
     <material>Gazebo/Grey</material>
   </gazebo>
   <gazebo reference="wheel_front_right">
-    <mul1>0.2</mul1>
-    <mul2>0.2</mul2>
+    <mul1>1.0</mul1>
+    <mul2>1.0</mul2>
+    <slip1>0.1</slip1>
+    <slip2>0.1</slip2>
     <material>Gazebo/Grey</material>
   </gazebo>
   <gazebo reference="wheel_rear_left">
-    <mul1>0.2</mul1>
-    <mul2>0.2</mul2>
+    <mul1>1.0</mul1>
+    <mul2>1.0</mul2>
+    <slip1>0.1</slip1>
+    <slip2>0.1</slip2>
     <material>Gazebo/Grey</material>
   </gazebo>
   <gazebo reference="wheel_rear_right">
-    <mul1>0.2</mul1>
-    <mul2>0.2</mul2>
+    <mul1>1.0</mul1>
+    <mul2>1.0</mul2>
+    <slip1>0.1</slip1>
+    <slip2>0.1</slip2>
     <material>Gazebo/Grey</material>
   </gazebo>
@@ -244,6 +258,6 @@
       <right_joint>wheel_rear_right_joint</right_joint>
       <!-- Kinematics -->
-      <wheel_separation>1.2</wheel_separation>
-      <wheel_separation>1.2</wheel_separation>
+      <wheel_separation>2.0</wheel_separation>
+      <wheel_separation>2.0</wheel_separation>
       <wheel_diameter>0.3</wheel_diameter>
       <wheel_diameter>0.3</wheel_diameter>
@@ -256,5 +270,5 @@
       <robot_base_frame>base_footprint</robot_base_frame>
       <max_wheel_torque>1000</max_wheel_torque>
-      <max_acceleration>20.0</max_acceleration>
+      <max_acceleration>30.0</max_acceleration>
     </plugin>
   </gazebo>

File: sim_ws/src/nav2_gps_waypoint_follower_demo/urdf/wheel_module_macro.xacro (robot description, xacro)
@@ -46,6 +46,6 @@
             <child link="wheel_module_${parent_name}"/>
             <origin xyz="${cx} ${cy} ${cz}" rpy="0 0 0"/> <!-- This origin is where child link is placed w.r.t parent link -->
-            <limit effort="1000" velocity="1000"/>
-            <dynamics damping="1.0" friction="1.0"/>
+            <!-- <limit effort="1000" velocity="1000"/> -->
+            <!-- <dynamics damping="1.0" friction="1.0"/> -->
         </joint>
         <!-- Define the wheel module link -->
@@ -83,6 +83,6 @@
             <origin xyz="0 ${wheel_position_y} ${-module_len/2.0}" rpy="0 0 0"/>
             <axis xyz="0 1 0"/>
-            <limit effort="1000" velocity="1000"/>
-            <dynamics damping="1.0" friction="1.0"/>
+            <limit effort="2000" velocity="2000"/>
+            <dynamics damping="1.0" friction="0.5"/>
         </joint>
         <link name="wheel_${parent_name}">
